File: pcb/KiCad Files/midi keyboard.kicad_pcb (KiCad board)
At the start: 2 copper layers, 211 x 121.5 mm, 50 parts, among them SW1 RotaryEncoder_Switch_MP, U1 Waveshare ESP32-S3-ZERO

Commit message: updated gerber files, finished schematic
Parts:
- added ?: LOGO, Hackclub Footprints:half-life-logo, F.Cu at (172.5, 54.0)
- added ?: LOGO, Hackclub Footprints:hack-club-logo, F.Cu at (112.5, 58.0)
